File: kicad/6-mic-array-pcb.kicad_pcb (KiCad board)
At the start: 4 copper layers, 100 x 120 mm, 11 parts, among them J1 USB-C-16P, U1 SF32LB52JUD6, U2 ADAU1977, U3 XC6206P332MR, U4 XC6206P332MR

Commit message: feat(common): add pdf
Parts:
- J1: footprint Connector_USB:USB_C_Receptacle_PCB -> Connector_USB:USB_C_Receptacle_Amphenol_12401548E4-2A
- MIC1, MIC2, MIC3, MIC4, MIC5, MIC6: footprint Microphone:MEMS_Mic_SMD_4.72x3.76mm -> Sensor_Audio:Knowles_LGA-6_4.72x3.76mm
- U1: footprint Package_LGA:LGA-56_6x6mm_P0.65mm -> 6-mic-array:SF32LB52JUD6_LGA56
- U3, U4: footprint Package_TO_SOT_SMD:SOT-23 -> Package_TO_SOT_SMD:SOT-23-3
- moved U3 65.0 mm to (155.0, 60.0)
- moved U4 65.0 mm to (155.0, 40.0)
- moved J1 40.0 mm to (220.0, 80.0)
Other:
- board size 100 x 120 mm -> 260 x 130 mm
